File: Hardware/Monster_Moto_Shield.brd (EAGLE design)
At the start: 53.3 x 59.7 mm, 44 parts, among them Q1 FDD8580, Q2 FDD8580, U1 VNH2SP30, U2 VNH2SP30, U3 ARDUINO_SHIELDLABEL

Commit message: Commit bec of computer change
Parts:
- removed U$6: CREATIVE_COMMONS, SparkFun:CREATIVE_COMMONS
- added FRAME*: FRAME-LETTER, SparkFun-Aesthetics:CREATIVE_COMMONS
- U3: value ARDUINO_SHIELDLABEL -> ARDUINO_R3_SHIELD; device SparkFun:DUEMILANOVE_SHIELD -> SparkFun-Boards:UNO_R3_SHIELD
- moved JP4 45.7 mm to (3.81, 58.4)
- moved JP6 34.4 mm to (45.7, 3.81)
- moved C4 13.7 mm to (5.69, 1.68), turned to 0 degrees
- moved R15 13.7 mm to (12.4, 1.75), turned to 0 degrees
- moved R14 13.5 mm to (8.86, 1.73), turned to 0 degrees
- moved R8 7.49 mm to (9.70, 22.5)
- moved R7 6.74 mm to (7.65, 22.5)
- moved LED5 5.24 mm to (50.8, 53.3)
- moved LED4 5.12 mm to (48.9, 53.3)
- moved R19 5.08 mm to (47.0, 53.3)
- moved R17 4.79 mm to (9.70, 19.1)
- moved C1 2.87 mm to (5.61, 15.7), turned to 0 degrees
- moved R5 2.47 mm to (7.59, 15.7)
- moved R6 2.19 mm to (9.68, 15.6)
- moved R11 1.95 mm to (45.2, 33.7)
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Routing:
- net N$8: track 51.4 -> 68.3 mm
- net 5V: track 17.2 -> 34.2 mm, vias 1 -> 4
- net CS2: track 8.20 -> 16.1 mm
- net N$12: track 37.1 -> 29.6 mm
- net EN1: track 2.44 -> 8.27 mm
- net GND: track 10.8 -> 15.3 mm, vias 14 -> 13
- net VCC: track 281.4 -> 278.0 mm
- net N$9: track 60.2 -> 57.8 mm
- net N$7: track 27.0 -> 29.2 mm
- net N$3: track 9.21 -> 7.17 mm
- net N$14: track 2.59 -> 4.00 mm
- net OUTB2: track 78.2 -> 76.9 mm
- net N$16: track 2.71 -> 3.82 mm
- net OUTB1: track 85.2 -> 86.1 mm
- net CS1: track 8.20 -> 7.31 mm
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Other:
- board text added: "V10"
- board text removed: "11/3/10"

Commit message: Computer Change
Parts:
- added U$3: (no value), SparkFun-Aesthetics:OSHW-LOGO-M
- added U$4, U$6: (no value), Testing:STAND-OFF
- moved FRAME* 113.9 mm to (-3.28, -14.0)
- moved R20 16.8 mm to (35.8, 1.98)
- moved LED1 16.5 mm to (34.3, 1.98)
- moved R14 10.2 mm to (19.1, 1.96), turned to 90 degrees
- moved R15 5.24 mm to (17.6, 1.98), turned to 270 degrees
- moved C4 4.57 mm to (5.69, 6.25)
- moved JP4 3.81 mm to (7.62, 58.4)
- moved LED4 2.54 mm to (48.9, 55.9)
- moved LED5 2.54 mm to (50.8, 55.9)
- moved R19 2.54 mm to (47.0, 55.9)
- moved JP6 1.27 mm to (47.0, 3.81)
- moved R1 0.05 mm to (47.0, 22.9)
- moved R12 0.05 mm to (47.0, 20.3)
- moved R13 0.05 mm to (47.0, 21.6)
- moved R2 0.05 mm to (47.0, 24.1)
Routing:
- net VCC: track 278.0 -> 301.7 mm
- net CS2: track 16.1 -> 21.8 mm
- net OUTB2: track 76.9 -> 75.1 mm
- net N$8: track 68.3 -> 67.2 mm, vias 4 -> 6
- net N$18: track 1.42 -> 2.06 mm
Other:
- outline, holes or cut-outs redrawn
- board text added: "J. Lindblom and N. Bernstein"
- board text added: "Revised by: Patrick Alberts"

Commit message: Cleared Up Drc Isssues
Parts:
- C1, C4: device SparkFun:0402-CAP -> SparkFun-Capacitors:0603-CAP
- moved C1 2.95 mm to (7.96, 13.9), turned to 270 degrees
- moved LED4 1.98 mm to (47.3, 57.1), turned to 270 degrees
- moved R12 1.95 mm to (46.8, 18.4)
- moved R19 1.93 mm to (47.2, 54.0), turned to 270 degrees
- moved R5 1.90 mm to (6.38, 17.1), turned to 180 degrees
- moved R10 1.81 mm to (46.9, 13.4)
- moved R13 1.62 mm to (46.8, 20.0)
- moved R7 1.50 mm to (6.37, 21.7), turned to 180 degrees
- moved R3 1.43 mm to (46.8, 15.1)
- moved R1 1.28 mm to (46.8, 21.6)
- moved R16 1.22 mm to (6.43, 19.3), turned to 180 degrees
- moved LED5 1.19 mm to (50.6, 57.1), turned to 270 degrees
- moved R4 1.08 mm to (46.8, 16.7)
- moved R2 0.96 mm to (46.8, 23.2)
- moved C4 0.15 mm to (5.61, 6.38)
Routing:
- net N$16: track 3.81 -> 7.37 mm
- net GND: track 15.1 -> 12.6 mm, vias 13 -> 10
- net EN1: track 8.38 -> 6.27 mm
- net N$4: track 32.8 -> 34.6 mm
- net PWM2: track 4.18 -> 5.56 mm
- net INB1: track 3.96 -> 5.33 mm
- net EN2: track 6.69 -> 5.32 mm
- net 5V: track 34.3 -> 33.0 mm, vias 4 -> 2
- net CS1: track 7.31 -> 8.59 mm
- net N$12: track 29.6 -> 30.8 mm
- net OUTB2: track 75.1 -> 74.0 mm
- net PWM1: track 4.23 -> 5.22 mm
- net INA2: track 2.96 -> 3.83 mm
- net N$2: track 58.5 -> 57.7 mm
- net INA1: track 2.91 -> 3.70 mm
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
Commit message: Added SF Flame, Cleaned Up SCH, Added Input v silk.
Parts:
- added LOGO1: SFE_LOGO_FLAME.2_INCH, SparkFun-Aesthetics:SFE_LOGO_FLAME_.2
Other:
- board text added: "Input 6-30V"
Changed lines of the file:
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@@
 <text x="26.8478" y="-14.097" size="1.778" layer="51" font="vector" ratio="10">J. Lindblom and N. Bernstein</text>
 <text x="8.2042" y="-17.1196" size="1.778" layer="51" font="vector" ratio="10">Revised by: Patrick Alberts</text>
+<text x="33.03778125" y="7.01548125" size="1.27" layer="21" font="vector" ratio="15" rot="R180">Input 6-30V</text>
 </plain>
 <attributes>
@@
 <element name="U$4" library="Testing" package="STAND-OFF" value="" x="7.62" y="2.54"/>
 <element name="U$6" library="Testing" package="STAND-OFF" value="" x="50.8" y="53.34"/>
+<element name="LOGO1" library="SparkFun-Aesthetics" package="SFE_LOGO_FLAME_.2" value="SFE_LOGO_FLAME.2_INCH" x="29.6037" y="24.846278125"/>
 </elements>
 <signals>

Commit message: Chaned LED res to 1k
Parts:
- removed R18, R19: 330, SparkFun-Resistors:0603
- added R21, R22: 1K, SparkFun-Resistors:0603-RES
- R20: value 330 -> 1K; device SparkFun-Resistors:0603 -> SparkFun-Resistors:0603-RES
- moved R20 0.06 mm to (35.8, 2.03), turned to 90 degrees
Connections:
- net N$14: now also R21.2; no longer R18.1
- net N$16: now also R22.2; no longer R19.1
- net N$18: now also R20.2; no longer R20.1
- net OUTA1: now also R21.1; no longer R18.2
- net OUTA2: now also R22.1; no longer R19.2
- net VCC: now also R20.1; no longer R20.2
Changed lines of the file:
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@@
 <?xml version="1.0" encoding="utf-8"?>
 <!DOCTYPE eagle SYSTEM "eagle.dtd">
-<eagle version="6.5.0">
+<eagle version="6.4">
 <drawing>
 <settings>
@@
 <setting verticaltext="up"/>
 </settings>
-<grid distance="0.05" unitdist="inch" unit="inch" style="lines" multiple="1" display="yes" altdistance="0.0001" altunitdist="inch" altunit="inch"/>
+<grid distance="0.05" unitdist="inch" unit="inch" style="lines" multiple="1" display="yes" altdistance="0.005" altunitdist="inch" altunit="inch"/>
 <layers>
 <layer number="1" name="Top" color="4" fill="1" visible="yes" active="yes"/>
@@
 <layer number="27" name="tValues" color="7" fill="1" visible="no" active="yes"/>
 <layer number="28" name="bValues" color="7" fill="1" visible="no" active="yes"/>
-<layer number="29" name="tStop" color="7" fill="3" visible="yes" active="yes"/>
+<layer number="29" name="tStop" color="7" fill="3" visible="no" active="yes"/>
 <layer number="30" name="bStop" color="7" fill="6" visible="no" active="yes"/>
 <layer number="31" name="tCream" color="7" fill="4" visible="no" active="yes"/>
@@
 <attribute name="VALUE" value="GREEN" x="50.634896875" y="57.0611" size="1.778" layer="27" rot="R270" display="off"/>
 </element>
-<element name="R18" library="SparkFun-Resistors" package="0603" value="330" x="2.54" y="48.26" rot="R90">
-<attribute name="PROD_ID" value="RES-08270" x="2.54" y="48.26" size="1.778" layer="27" rot="R90" display="off"/>
-<attribute name="VALUE" value="33OHM" x="2.54" y="48.26" size="1.778" layer="27" rot="R90" display="off"/>
-</element>
-<element name="R19" library="SparkFun-Resistors" package="0603" value="330" x="47.200821875" y="53.959765625" rot="R270">
-<attribute name="PROD_ID" value="RES-08270" x="47.200821875" y="53.959765625" size="1.778" layer="27" rot="R270" display="off"/>
-<attribute name="VALUE" value="33OHM" x="47.200821875" y="53.959765625" size="1.778" layer="27" rot="R270" display="off"/>
-</element>
-<element name="R20" library="SparkFun-Resistors" package="0603" value="330" x="35.8394" y="1.9812" smashed="yes" rot="R270">
-<attribute name="NAME" x="36.5379" y="2.8702" size="0.4064" layer="25" rot="R270"/>
-<attribute name="VALUE" value="33OHM" x="34.6964" y="3.0607" size="0.4064" layer="27" rot="R270"/>
-<attribute name="PROD_ID" value="RES-08270" x="35.8394" y="1.9812" size="1.778" layer="27" rot="R270" display="off"/>
-</element>
 <element name="JP5" library="SparkFun" package="SFE-NEW-WEBLOGO" value="LOGO-SFENEW" x="27.559" y="17.399" rot="MR90"/>
 <element name="U3" library="SparkFun-Boards" package="UNO_R3_SHIELD" value="ARDUINO_R3_SHIELD" x="53.34" y="59.69" rot="R180"/>
@@
 <element name="U$6" library="Testing" package="STAND-OFF" value="" x="50.8" y="53.34"/>
 <element name="LOGO1" library="SparkFun-Aesthetics" package="SFE_LOGO_FLAME_.2" value="SFE_LOGO_FLAME.2_INCH" x="29.6037" y="24.846278125"/>
+<element name="R20" library="SparkFun-Resistors" package="0603-RES" value="1K" x="35.814" y="2.032" rot="R90">
+<attribute name="PROD_ID" value="RES-07856" x="35.814" y="2.032" size="1.778" layer="27" font="vector" ratio="15" rot="R90" display="off"/>
+</element>
+<element name="R21" library="SparkFun-Resistors" package="0603-RES" value="1K" x="2.54" y="48.26" rot="R270">
+<attribute name="PROD_ID" value="RES-07856" x="2.54" y="48.26" size="1.778" layer="27" font="vector" ratio="15" rot="R270" display="off"/>
+</element>
+<element name="R22" library="SparkFun-Resistors" package="0603-RES" value="1K" x="47.244" y="54.229" rot="R90">
+<attribute name="PROD_ID" value="RES-07856" x="47.244" y="54.229" size="1.778" layer="27" font="vector" ratio="15" rot="R90" display="off"/>
+</element>
 </elements>
 <signals>
 <signal name="OUTA1">
 <contactref element="JP1" pad="1"/>
-<contactref element="R18" pad="2"/>
 <contactref element="U1" pad="1"/>
 <contactref element="U1" pad="30"/>
@@
 <wire x1="6.35" y1="57.15" x2="2.54" y2="53.34" width="0.254" layer="16"/>
 <wire x1="15.24" y1="57.15" x2="6.35" y2="57.15" width="0.254" layer="16"/>
-<wire x1="2.54" y1="52.07" x2="2.54" y2="49.11" width="0.254" layer="1"/>
 <via x="2.54" y="52.07" extent="1-16" drill="0.508"/>
 <wire x1="2.54" y1="53.34" x2="2.54" y2="52.07" width="0.254" layer="16"/>
+<contactref element="R21" pad="1"/>
+<wire x1="2.54" y1="49.11" x2="2.54" y2="52.07" width="0.254" layer="1"/>
 </signal>
 <signal name="OUTB1">
@@
 <contactref element="C5" pad="+"/>
 <contactref element="C6" pad="1"/>
-<contactref element="R20" pad="2"/>
 <contactref element="U1" pad="13"/>
 <contactref element="U1" pad="3"/>
@@
 <wire x1="38.1" y1="5.08" x2="38.1" y2="2.499359375" width="0.254" layer="1"/>
 <wire x1="38.1" y1="2.499359375" x2="36.751259375" y2="1.15061875" width="0.254" layer="1"/>
-<wire x1="36.751259375" y1="1.15061875" x2="35.85881875" y2="1.15061875" width="0.254" layer="1"/>
-<wire x1="35.85881875" y1="1.15061875" x2="35.8394" y2="1.1312" width="0.254" layer="1"/>
+<contactref element="R20" pad="1"/>
+<wire x1="36.751259375" y1="1.15061875" x2="35.84538125" y2="1.15061875" width="0.254" layer="1"/>
+<wire x1="35.84538125" y1="1.15061875" x2="35.814" y2="1.182" width="0.254" layer="1"/>
 </signal>
 <signal name="N$1">
@@
 <signal name="OUTA2">
 <contactref element="JP2" pad="1"/>
-<contactref element="R19" pad="2"/>
 <contactref element="U2" pad="1"/>
 <contactref element="U2" pad="30"/>
@@
 <wire x1="43.54321875" y1="54.991" x2="47.190659375" y2="51.343559375" width="0.254" layer="16"/>
 <via x="47.190659375" y="51.343559375" extent="1-16" drill="0.508"/>
-<wire x1="47.190659375" y1="51.343559375" x2="47.190659375" y2="53.099603125" width="0.254" layer="1"/>
-<wire x1="47.190659375" y1="53.099603125" x2="47.200821875" y2="53.109765625" width="0.254" layer="1"/>
+<contactref element="R22" pad="1"/>
+<wire x1="47.190659375" y1="51.343559375" x2="47.190659375" y2="53.325659375" width="0.254" layer="1"/>
+<wire x1="47.190659375" y1="53.325659375" x2="47.244" y2="53.379" width="0.254" layer="1"/>
 </signal>
 <signal name="N$16">
 <contactref element="LED4" pad="A"/>
 <contactref element="LED5" pad="C"/>
-<contactref element="R19" pad="1"/>
-<wire x1="46.427959375" y1="57.0585625" x2="47.200821875" y2="56.2857" width="0.254" layer="1"/>
-<wire x1="47.200821875" y1="56.2857" x2="47.200821875" y2="55.88" width="0.254" layer="1"/>
-<wire x1="47.200821875" y1="55.88" x2="47.200821875" y2="54.809765625" width="0.254" layer="1"/>
-<wire x1="51.511896875" y1="57.0611" x2="50.330796875" y2="55.88" width="0.254" layer="1"/>
-<wire x1="50.330796875" y1="55.88" x2="47.200821875" y2="55.88" width="0.254" layer="1"/>
+<contactref element="R22" pad="2"/>
+<wire x1="51.511896875" y1="57.0611" x2="51.511896875" y2="56.464896875" width="0.254" layer="1"/>
+<wire x1="51.511896875" y1="56.464896875" x2="51.308" y2="56.261" width="0.254" layer="1"/>
+<wire x1="51.308" y1="56.261" x2="47.244" y2="56.261" width="0.254" layer="1"/>
+<wire x1="46.99" y1="56.261" x2="46.609" y2="56.261" width="0.254" layer="1"/>
+<wire x1="46.609" y1="56.261" x2="46.482" y2="56.388" width="0.254" layer="1"/>
+<wire x1="46.482" y1="56.388" x2="46.482" y2="57.004521875" width="0.254" layer="1"/>
+<wire x1="46.482" y1="57.004521875" x2="46.427959375" y2="57.0585625" width="0.254" layer="1"/>
+<wire x1="47.244" y1="55.079" x2="47.244" y2="56.261" width="0.254" layer="1"/>
+<wire x1="47.244" y1="56.261" x2="46.99" y2="56.261" width="0.254" layer="1"/>
 </signal>
 <signal name="N$18">
 <contactref element="LED1" pad="A"/>
-<contactref element="R20" pad="1"/>
-<wire x1="34.3408" y1="2.8582" x2="35.8124" y2="2.8582" width="0.254" layer="1"/>
-<wire x1="35.8124" y1="2.8582" x2="35.8394" y2="2.8312" width="0.254" layer="1"/>
+<contactref element="R20" pad="2"/>
+<wire x1="34.3408" y1="2.8582" x2="35.7902" y2="2.8582" width="0.254" layer="1"/>
+<wire x1="35.7902" y1="2.8582" x2="35.814" y2="2.882" width="0.254" layer="1"/>
 </signal>
 <signal name="N$14">
 <contactref element="LED2" pad="A"/>
 <contactref element="LED3" pad="C"/>
-<contactref element="R18" pad="1"/>
-<wire x1="2.54" y1="47.41" x2="2.64" y2="47.51" width="0.254" layer="1"/>
 <wire x1="4.445" y1="47.3322" x2="6.2992" y2="47.3322" width="0.254" layer="1"/>
 <wire x1="6.2992" y1="47.3322" x2="6.35" y2="47.383" width="0.254" layer="1"/>
-<wire x1="4.445" y1="47.3322" x2="2.6178" y2="47.3322" width="0.254" layer="1"/>
-<wire x1="2.6178" y1="47.3322" x2="2.54" y2="47.41" width="0.254" layer="1"/>
+<contactref element="R21" pad="2"/>
+<wire x1="4.445" y1="47.3322" x2="4.445" y2="47.41" width="0.254" layer="1"/>
+<wire x1="4.445" y1="47.41" x2="2.54" y2="47.41" width="0.254" layer="1"/>
 </signal>
 </signals>
